Commit message: fix: 修复了haerdwareinterface插件中的函数签名错误 test: 修复了test中的小问题

File: dji_motor_hardwear_interface/test/config/test_robot.ros2_control.xacro (robot description, xacro)
@@ -1,19 +1,19 @@
 <?xml version="1.0"?>
 <robot xmlns:xacro="http://www.ros.org/wiki/xacro">
-        <ros2_control name="dji_motor_hardwear_interface_test_robot_control" type="system">
-            <hardware>
-                <plugin>RM_hardware_interface/RM_DJIMotorHardwareInterface</plugin>
-                <param name="command_frequence">1000</param>
-                <param name="can_port">can0</param>
-            </hardware>
-            <joint name="GM6020_test_joint">
-                <param name="can_id">1</param>
-                <param name="motor_type">GM6020</param>
-                <command_interface name="moment"/>
-                <state_interface name="position"/>
-                <state_interface name="velocity"/>
-                <state_interface name="moment"/>
-                <state_interface name="temperature"/>
-            </joint>
-        </ros2_control>
+    <ros2_control name="test_robot_control" type="system">
+        <hardware>
+            <plugin>RM_hardware_interface/RM_DJIMotorHardwareInterface</plugin>
+            <param name="command_frequence">1000</param>
+            <param name="can_port">can0</param>
+        </hardware>
+        <joint name="GM6020_test_joint">
+            <param name="can_id">1</param>
+            <param name="motor_type">GM6020</param>
+            <command_interface name="moment"/>
+            <state_interface name="position"/>
+            <state_interface name="velocity"/>
+            <state_interface name="moment"/>
+            <state_interface name="temperature"/>
+        </joint>
+    </ros2_control>
 </robot>

File: dji_motor_hardwear_interface/test/config/test_robot.urdf.xacro (robot description, xacro)
@@ -2,5 +2,5 @@
 <robot xmlns:xacro="http://www.ros.org/wiki/xacro" name="test_robot">
     <!-- Import test_robot urdf file -->
-    <xacro:include filename="$(find dji_motor_hardwear_interface)/test/config/test_robot.urdf" />
+    <xacro:include filename="test_robot.urdf" />
     <!-- Import control_xacro -->
     <xacro:include filename="test_robot.ros2_control.xacro" />
