Commit message: feature: 添加了 C610 电机的支持 test: 在测试配置中添加了 C610 电机

File: core/dji_motor_hardwear_interface/test/config/test_robot.ros2_control.xacro (robot description, xacro)
@@ -7,5 +7,5 @@
             <param name="can_port">can0</param>
         </hardware>
-        <joint name="GM6020_test_joint">
+        <joint name="GM6020_joint">
             <param name="can_id">1</param>
             <param name="motor_type">GM6020</param>
@@ -16,4 +16,21 @@
             <state_interface name="temperature"/>
         </joint>
+        <joint name="C620_joint">
+            <param name="can_id">2</param>
+            <param name="motor_type">C620</param>
+            <command_interface name="moment"/>
+            <state_interface name="position"/>
+            <state_interface name="velocity"/>
+            <state_interface name="moment"/>
+            <state_interface name="temperature"/>
+        </joint>
+        <joint name="C610_joint">
+            <param name="can_id">3</param>
+            <param name="motor_type">C610</param>
+            <command_interface name="moment"/>
+            <state_interface name="position"/>
+            <state_interface name="velocity"/>
+            <state_interface name="moment"/>
+        </joint>
     </ros2_control>
 </robot>

File: core/dji_motor_hardwear_interface/test/config/test_robot.urdf (robot description, URDF)
Before this commit: robot test_robot, 2 links, 1 joints
Links:
- added link link_2; visual cylinder length=0.5 radius=0.05
- added link link_3; visual cylinder length=0.5 radius=0.05
Joints:
- removed joint GM6020_test_joint
- added joint C610_joint: type revolute, parent link_2, child link_3, origin xyz=0 0 0.25 rpy=0 0 0, axis 1 0 0, limit lower=-1.57 upper=1.57 effort=1 velocity=1
- added joint C620_joint: type revolute, parent link_1, child link_2, origin xyz=0 0 0.25 rpy=0 0 0, axis 0 1 0, limit lower=-1.57 upper=1.57 effort=1 velocity=1
- added joint GM6020_joint: type revolute, parent base_link, child link_1, origin xyz=0 0 0.25 rpy=0 0 0, axis 0 0 1, limit lower=-1.57 upper=1.57 effort=1 velocity=1
